File: ultrasonic_roborio.sch (KiCad schematic (older format))
At the start: 16 parts, among them J1 PCM solenoid, J2 Sensor0, J3 roboRIO A0, J4 Sensor1, J5 roboRIO A1, SW0 SW_Push, SW1 SW_Push, SW2 SW_Push, SW3 SW_Push

Commit message: Initial work on tracing
Parts:
- renumbered SW1 to SW0, SW0 to SW1
Changed lines of the file:
@@
 	5950 1900 5950 1950
 $Comp
-L Switch:SW_Push SW1
+L Switch:SW_Push SW0
 U 1 1 5E529459
 P 5700 1500
-F 0 "SW1" H 5700 1693 50  0000 C CNN
+F 0 "SW0" H 5700 1693 50  0000 C CNN
 F 1 "SW_Push" H 5700 1694 50  0001 C CNN
 F 2 "Button_Switch_THT:SW_PUSH_6mm" H 5700 1700 50  0001 C CNN
@@
 $EndComp
 $Comp
-L Switch:SW_Push SW0
+L Switch:SW_Push SW1
 U 1 1 5E527FD3
 P 5700 1900
-F 0 "SW0" H 5700 2093 50  0000 C CNN
+F 0 "SW1" H 5700 2093 50  0000 C CNN
 F 1 "SW_Push" H 5700 2094 50  0001 C CNN
 F 2 "Button_Switch_THT:SW_PUSH_6mm" H 5700 2100 50  0001 C CNN

Commit message: Finish v0 PCB design Add protection resistor for if A1 and A2 pressed at the same time Change layout to reduce board size Move buttons to not have wires running over them (risk of accidential triggering) Add author names This commit has the gerbers that were ordered as the ZIP file
Parts:
- added R1: 330, Resistor_SMD:R_0603_1608Metric, symbol Device:R
- J1: footprint ultrasonic_roborio:LSF-SMT 3.50_02_135 3.5SN -> ultrasonic_roborio:LSF-SMT_3.50_02_135_3.5SN
- J2, J4: footprint ultrasonic_roborio:LSF-SMT 3.50_04_135 3.5SN -> ultrasonic_roborio:LSF-SMT_3.50_04_135_3.5SN
- SW1: renamed from SW0; footprint Button_Switch_THT:SW_PUSH_6mm -> Button_Switch_SMD:SW_SPST_PTS810
- SW2: renamed from SW1; footprint Button_Switch_THT:SW_PUSH_6mm -> Button_Switch_SMD:SW_SPST_PTS810
- SW3: renamed from SW2; footprint Button_Switch_THT:SW_PUSH_6mm -> Button_Switch_SMD:SW_SPST_PTS810
- SW4: renamed from SW3; footprint Button_Switch_THT:SW_PUSH_6mm -> Button_Switch_SMD:SW_SPST_PTS810
- renumbered JP2 to JP1, JP1 to JP2, R1 to R2, R2 to R3, R3 to R4, R4 to R5
Connections:
- net +24V: now also R1.1; no longer SW1.2, SW3.2
- new net TeachV+: R1.2, SW1.2, SW3.2
